File: IRQF103C8.brd (EAGLE design)
At the start: 70 x 40 mm, 64 parts, among them IC1 STM32F10XCXT6, IC2 LM1117IMPX-3.3, IC3 LM1117MPX-5.0, Q1 8MHz, Q2 32.768kHz, Q3 BC817-40SMD, U1 USBUF02W6

Commit message: Update files
Update schematic & pcb files
Parts:
- added C8: (no value), cap-master:3216/T
- added R2: 910k, resistor:M0805
- moved L2 1.60 mm to (46.9, 24.4)
- moved C7 0.20 mm to (42.9, 24.2)
Connections:
- net GND: now also C8.-
- net N$3: now also R2.2
- net N$4: now also R2.1
- net VDDA: now also C8.+
Routing:
- net N$4: track 14.8 -> 18.3 mm
- net N$3: track 17.3 -> 20.6 mm
- net VDDA: track 6.23 -> 8.08 mm
- net GND: vias 71 -> 68
Changed lines of the file:
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@@
 <setting verticaltext="up"/>
 </settings>
-<grid distance="0.1" unitdist="mm" unit="mm" style="lines" multiple="1" display="yes" altdistance="0.025" altunitdist="inch" altunit="mm"/>
+<grid distance="0.2" unitdist="mm" unit="mm" style="lines" multiple="1" display="yes" altdistance="0.025" altunitdist="inch" altunit="mm"/>
 <layers>
 <layer number="1" name="Top" color="4" fill="1" visible="yes" active="yes"/>
@@
 <attribute name="VALUE" x="34.6805" y="-31.151" size="0.8128" layer="48" font="vector" ratio="15" rot="R180"/>
 </element>
-<element name="C7" library="cap-master" package="0805" value="100n" x="43.1" y="24.234" smashed="yes" rot="R90">
-<attribute name="NAME" x="41.0525" y="26.2185" size="1.016" layer="25" font="vector" ratio="15" rot="R270"/>
-<attribute name="VALUE" x="37.4185" y="-29.295" size="0.8128" layer="48" font="vector" ratio="15" rot="R180"/>
+<element name="C7" library="cap-master" package="0805" value="100n" x="42.9" y="24.234" smashed="yes" rot="R90">
+<attribute name="NAME" x="40.8525" y="26.2185" size="1.016" layer="25" font="vector" ratio="15" rot="R270"/>
+<attribute name="VALUE" x="37.2185" y="-29.295" size="0.8128" layer="48" font="vector" ratio="15" rot="R180"/>
 </element>
 <element name="IC1" library="stm32" package="TQFP48" value="STM32F10XCXT6" x="35.806" y="20.242" smashed="yes" rot="R90">
@@
 <attribute name="VALUE" x="29.676" y="17.302" size="1.016" layer="21" font="vector" ratio="15" rot="R90"/>
 </element>
-<element name="L2" library="ipc-7351-inductor" package="INDC1608X95N" value="10uH" x="45.3" y="24.446" smashed="yes" rot="R90">
-<attribute name="NAME" x="47.1825" y="24.471" size="1.016" layer="25" font="vector" ratio="15" rot="R90"/>
-<attribute name="VALUE" x="41.271" y="-33.2875" size="0.8128" layer="48" font="vector" ratio="15"/>
+<element name="L2" library="ipc-7351-inductor" package="INDC1608X95N" value="10uH" x="46.9" y="24.446" smashed="yes" rot="R90">
+<attribute name="NAME" x="48.7825" y="24.471" size="1.016" layer="25" font="vector" ratio="15" rot="R90"/>
+<attribute name="VALUE" x="42.871" y="-33.2875" size="0.8128" layer="48" font="vector" ratio="15"/>
 </element>
 <element name="LD6" library="led" package="CHIPLED_0805" value="" x="27.904" y="36.184" smashed="yes" rot="R90">
@@
 <attribute name="NAME" x="64.3138" y="20.6288" size="1.016" layer="25" font="vector" ratio="15"/>
 <attribute name="VALUE" x="60.99" y="20.025" size="1.27" layer="27"/>
+</element>
+<element name="R2" library="resistor" package="M0805" value="910k" x="53" y="21.6" smashed="yes" rot="MR90">
+<attribute name="NAME" x="54.016" y="23.716" size="1.016" layer="26" font="vector" ratio="15" rot="MR0"/>
+<attribute name="VALUE" x="50.714" y="20.584" size="1.27" layer="48" rot="MR90"/>
+</element>
+<element name="C8" library="cap-master" package="3216/T" value="" x="44.9" y="24.7" smashed="yes" rot="R270">
+<attribute name="NAME" x="42.97" y="28.0875" size="1.016" layer="25" font="vector" ratio="15" rot="R270"/>
+<attribute name="VALUE" x="42.6775" y="26.2875" size="0.8128" layer="27" ratio="10" rot="R270"/>
 </element>
 </elements>
@@
 <wire x1="48.592" y1="19.992" x2="50.846" y2="22.246" width="0.254" layer="1"/>
 <wire x1="50.846" y1="22.246" x2="50.846" y2="24.001" width="0.254" layer="1"/>
+<contactref element="R2" pad="2"/>
+<wire x1="53" y1="22.55" x2="53" y2="23.4" width="0.254" layer="16"/>
+<wire x1="53" y1="23.4" x2="52.399" y2="24.001" width="0.254" layer="16"/>
+<wire x1="52.399" y1="24.001" x2="50.846" y2="24.001" width="0.254" layer="16"/>
 </signal>
 <signal name="N$4">
@@
 <wire x1="40.306" y1="19.492" x2="50.529" y2="19.492" width="0.254" layer="1"/>
 <wire x1="50.529" y1="19.492" x2="50.846" y2="19.175" width="0.254" layer="1"/>
+<contactref element="R2" pad="1"/>
+<wire x1="53" y1="20.65" x2="52.9" y2="20.55" width="0.254" layer="16"/>
+<wire x1="52.9" y1="20.55" x2="52.9" y2="19.4" width="0.254" layer="16"/>
+<wire x1="52.9" y1="19.4" x2="52.675" y2="19.175" width="0.254" layer="16"/>
+<wire x1="52.675" y1="19.175" x2="50.846" y2="19.175" width="0.254" layer="16"/>
 </signal>
 <signal name="NRST">
@@
 <wire x1="26.6" y1="27.2" x2="27.5395" y2="26.2605" width="0.4064" layer="16"/>
 <wire x1="27.5395" y1="26.2605" x2="29.4" y2="26.2605" width="0.4064" layer="16"/>
-<via x="44.4" y="27.4" extent="1-16" drill="0.4"/>
+<via x="44.4" y="28.2" extent="1-16" drill="0.4"/>
 <wire x1="29.37236875" y1="21.6" x2="29.371128125" y2="21.598759375" width="0.254" layer="16"/>
 <wire x1="26.966" y1="33.966" x2="26.966" y2="34.062" width="0.3048" layer="1"/>
@@
 <wire x1="41" y1="20.8" x2="41.6" y2="21.4" width="0.254" layer="16"/>
 <wire x1="41.6" y1="21.4" x2="41.6" y2="25.4" width="0.254" layer="16"/>
-<wire x1="41.6" y1="25.4" x2="43.6" y2="27.4" width="0.254" layer="16"/>
-<wire x1="43.6" y1="27.4" x2="44.4" y2="27.4" width="0.254" layer="16"/>
-<wire x1="44.4" y1="27.4" x2="45.3" y2="26.5" width="0.254" layer="1"/>
-<wire x1="45.3" y1="26.5" x2="45.3" y2="25.246" width="0.254" layer="1"/>
 <wire x1="48.6" y1="27" x2="47.2" y2="27" width="0.254" layer="1"/>
-<wire x1="47.2" y1="27" x2="46.6" y2="26.4" width="0.254" layer="1"/>
-<wire x1="46.6" y1="26.4" x2="46.6" y2="25.6" width="0.254" layer="1"/>
-<wire x1="46.6" y1="25.6" x2="46.246" y2="25.246" width="0.254" layer="1"/>
-<wire x1="46.246" y1="25.246" x2="45.3" y2="25.246" width="0.254" layer="1"/>
 <wire x1="15.4" y1="19.8" x2="17.6" y2="17.6" width="0.3048" layer="16"/>
 <wire x1="17.6" y1="17.6" x2="18.2" y2="17.6" width="0.3048" layer="16"/>
@@
 <wire x1="64.2" y1="14.2" x2="62.26" y2="16.14" width="0.254" layer="16"/>
 <wire x1="62.26" y1="16.14" x2="62.26" y2="17" width="0.254" layer="16"/>
+<wire x1="41.6" y1="25.4" x2="44.4" y2="28.2" width="0.254" layer="16"/>
+<wire x1="44.4" y1="28.2" x2="46" y2="28.2" width="0.254" layer="1"/>
+<wire x1="46" y1="28.2" x2="47.2" y2="27" width="0.254" layer="1"/>
+<wire x1="46.9" y1="25.246" x2="48.6" y2="26.946" width="0.254" layer="1"/>
+<wire x1="48.6" y1="26.946" x2="48.6" y2="27" width="0.254" layer="1"/>
 </signal>
 <signal name="N$19">
@@
 <contactref element="C7" pad="1"/>
 <wire x1="40.306" y1="21.492" x2="41.892" y2="21.492" width="0.254" layer="1"/>
-<wire x1="41.892" y1="21.492" x2="42.2" y2="21.8" width="0.254" layer="1"/>
-<wire x1="42.2" y1="21.8" x2="42.2" y2="22.3815" width="0.254" layer="1"/>
-<wire x1="42.2" y1="22.3815" x2="43.1" y2="23.2815" width="0.254" layer="1"/>
-<wire x1="45.3" y1="23.646" x2="44.9355" y2="23.2815" width="0.254" layer="1"/>
-<wire x1="44.9355" y1="23.2815" x2="43.1" y2="23.2815" width="0.254" layer="1"/>
+<contactref element="C8" pad="+"/>
+<wire x1="41.892" y1="21.492" x2="42.9" y2="22.5" width="0.254" layer="1"/>
+<wire x1="42.9" y1="22.5" x2="42.9" y2="23.2815" width="0.254" layer="1"/>
+<wire x1="42.9" y1="23.2815" x2="43.069" y2="23.1125" width="0.254" layer="1"/>
+<wire x1="43.069" y1="23.1125" x2="44.9" y2="23.1125" width="0.254" layer="1"/>
+<wire x1="46.9" y1="23.646" x2="46.3665" y2="23.1125" width="0.254" layer="1"/>
+<wire x1="46.3665" y1="23.1125" x2="44.9" y2="23.1125" width="0.254" layer="1"/>
 </signal>
 <signal name="DP">
@@
 <via x="23.6" y="19.4" extent="1-16" drill="0.4"/>
 <via x="56.2" y="19.8" extent="1-16" drill="0.4"/>
-<via x="53.2" y="21.6" extent="1-16" drill="0.4"/>
-<via x="52.6" y="23.8" extent="1-16" drill="0.4"/>
-<via x="49.6" y="22.8" extent="1-16" drill="0.4"/>
+<via x="48.2" y="22.8" extent="1-16" drill="0.4"/>
 <via x="33.4" y="19.8" extent="1-16" drill="0.4"/>
 <via x="34.8" y="17.6" extent="1-16" drill="0.4"/>
-<via x="43.4" y="21.6" extent="1-16" drill="0.4"/>
 <via x="41.6" y="12.2" extent="1-16" drill="0.4"/>
 <via x="48.2" y="12" extent="1-16" drill="0.4"/>
@@
 <via x="47.6" y="21" extent="1-16" drill="0.4"/>
 <via x="50" y="26.4" extent="1-16" drill="0.4"/>
-<via x="47.6" y="25.6" extent="1-16" drill="0.4"/>
 <via x="53.4" y="29" extent="1-16" drill="0.4"/>
 <via x="60.4" y="8.2" extent="1-16" drill="0.4"/>
@@
 <via x="25.8" y="14.4" extent="1-16" drill="0.4"/>
 <contactref element="C6" pad="-"/>
-<via x="47.6" y="23.2" extent="1-16" drill="0.4"/>
 <via x="53" y="26.4" extent="1-16" drill="0.4"/>
-<via x="47" y="28.4" extent="1-16" drill="0.4"/>
+<via x="47.2" y="28.4" extent="1-16" drill="0.4"/>
 <via x="42.8" y="28.2" extent="1-16" drill="0.4"/>
 <contactref element="JP1" pad="12"/>
@@
 <contactref element="BOOT0" pad="3"/>
 <contactref element="BOOT1" pad="3"/>
+<contactref element="C8" pad="-"/>
+<via x="48.6" y="25.2" extent="1-16" drill="0.4"/>
+<via x="43.4" y="21.6" extent="1-16" drill="0.4"/>
 <wire x1="33" y1="22.8" x2="33.556" y2="24.742" width="0" layer="19" extent="1-1"/>
 <wire x1="31.306" y1="17.992" x2="33.4" y2="19.8" width="0" layer="19" extent="1-1"/>
