File: IRQF103C8.sch (EAGLE design)
At the start: 62 parts, among them IC1 STM32F10XCXT6, IC2 LM1117IMPX-3.3, IC3 LM1117MPX-5.0, Q1 8MHz, Q2 32.768kHz, Q3 BC817-40SMD, U1 USBUF02W6

Commit message: Update files
Update schematic & pcb files
Parts:
- added C8: (no value), cap-master:CP-3216
- added R2: 910k, resistor:R-US_M0805
Connections:
- net GND: now also C8.-
- net N$3: now also R2.2
- net N$4: now also R2.1
- net VDDA: now also C8.+
Changed lines of the file:
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@@
 <part name="BOOT0" library="pinhead" deviceset="PINHD-1X3" device=""/>
 <part name="BOOT1" library="pinhead" deviceset="PINHD-1X3" device=""/>
+<part name="R2" library="resistor" deviceset="R-US_" device="M0805" value="910k"/>
+<part name="C8" library="cap-master" deviceset="CP-" device="3216"/>
 </parts>
 <sheets>
@@
 <instance part="BOOT0" gate="A" x="370.84" y="190.5"/>
 <instance part="BOOT1" gate="A" x="370.84" y="223.52"/>
+<instance part="R2" gate="G$1" x="66.04" y="88.9" rot="R270"/>
+<instance part="C8" gate="G$1" x="78.74" y="68.58" rot="R90"/>
 </instances>
 <busses>
@@
 <junction x="71.12" y="96.52"/>
 <pinref part="C4" gate="G$1" pin="1"/>
+<pinref part="R2" gate="G$1" pin="2"/>
+<wire x1="66.04" y1="83.82" x2="71.12" y2="83.82" width="0.1524" layer="91"/>
+<wire x1="71.12" y1="83.82" x2="71.12" y2="96.52" width="0.1524" layer="91"/>
 </segment>
 </net>
@@
 <wire x1="63.5" y1="99.06" x2="63.5" y2="106.68" width="0.1524" layer="91"/>
 <pinref part="Q1" gate="G$1" pin="2"/>
-<wire x1="63.5" y1="106.68" x2="71.12" y2="106.68" width="0.1524" layer="91"/>
+<wire x1="63.5" y1="106.68" x2="66.04" y2="106.68" width="0.1524" layer="91"/>
+<wire x1="66.04" y1="106.68" x2="71.12" y2="106.68" width="0.1524" layer="91"/>
 <wire x1="71.12" y1="106.68" x2="71.12" y2="104.14" width="0.1524" layer="91"/>
 <wire x1="76.2" y1="106.68" x2="71.12" y2="106.68" width="0.1524" layer="91"/>
 <junction x="71.12" y="106.68"/>
 <pinref part="C3" gate="G$1" pin="1"/>
+<pinref part="R2" gate="G$1" pin="1"/>
+<wire x1="66.04" y1="93.98" x2="66.04" y2="106.68" width="0.1524" layer="91"/>
+<junction x="66.04" y="106.68"/>
 </segment>
 </net>
@@
 <wire x1="68.58" y1="71.12" x2="68.58" y2="73.66" width="0.1524" layer="91"/>
 <junction x="68.58" y="73.66"/>
+<pinref part="C8" gate="G$1" pin="+"/>
+<wire x1="78.74" y1="71.12" x2="78.74" y2="73.66" width="0.1524" layer="91"/>
 </segment>
 <segment>
@@
 <pinref part="GND34" gate="1" pin="GND"/>
 <pinref part="C7" gate="G$1" pin="2"/>
-<wire x1="68.58" y1="66.04" x2="68.58" y2="60.96" width="0.1524" layer="91"/>
-</segment>
-<segment>
+<wire x1="68.58" y1="66.04" x2="68.58" y2="63.5" width="0.1524" layer="91"/>
+<pinref part="C8" gate="G$1" pin="-"/>
+<wire x1="68.58" y1="63.5" x2="68.58" y2="60.96" width="0.1524" layer="91"/>
+<wire x1="78.74" y1="66.04" x2="78.74" y2="63.5" width="0.1524" layer="91"/>
+<wire x1="78.74" y1="63.5" x2="68.58" y2="63.5" width="0.1524" layer="91"/>
+<junction x="68.58" y="63.5"/>
+</segment>
+<segment>
