File: Eagle/rev. B/IRQF103C8revB.brd (EAGLE design)
At the start: 70 x 40 mm, 66 parts, among them IC1 STM32F10XCXT6, IC2 LM1117IMPX-3.3, IC3 LM1117MPX-5.0, Q1 8MHz, Q2 32.768kHz, Q3 BC817-40SMD, U1 USBUF02W6

Commit message: refresh
Refresh and update files
Parts:
- removed C8: (no value), cap-master:3216/T
- moved Q2 4.08 mm to (45.8, 14.8)
- moved C1 3.82 mm to (49.1, 14.7)
- moved C2 3.82 mm to (49.1, 12.7)
- moved L2 3.21 mm to (43.7, 24.8), flipped to the bottom, turned to 270 degrees
- moved R2 2.01 mm to (51.0, 21.4)
- moved Q1 2.01 mm to (48.8, 21.4)
- moved C7 1.84 mm to (41.7, 25.6), flipped to the bottom
- moved C3 1.81 mm to (52.7, 19.3)
- moved C4 1.81 mm to (52.7, 24.1)
- moved C18 1.60 mm to (42.2, 15.8), turned to 270 degrees
Connections:
- net GND: no longer C8.-
- net VDDA: no longer C8.+
Routing:
- net PC13: track 40.8 -> 46.3 mm
- net GND: track 5.89 -> 11.4 mm, vias 68 -> 61
- net +3V3: track 211.0 -> 205.6 mm, vias 10 -> 8
- net NRST: track 64.8 -> 68.9 mm
- net N$1: track 15.3 -> 11.4 mm
- net N$2: track 13.4 -> 9.64 mm
- net N$4: track 18.3 -> 15.6 mm
- net N$3: track 20.6 -> 18.0 mm
- net PA10: track 11.7 -> 12.6 mm
- net VDDA: track 8.08 -> 7.30 mm, vias 0 -> 1
- net PA11: track 19.1 -> 19.8 mm
- net PA12: track 19.1 -> 19.7 mm
Other:
- board text added: "v.1.006 rev. B"
- board text removed: "v.1.006 rev. A"
