File: Eagle/rev. D/IRQF103C8revC.brd (EAGLE design)
At the start: 70 x 40 mm, 68 parts, among them IC1 STM32F10XCXT6, IC2 LM1117IMPX-3.3, IC3 LM1117MPX-5.0, Q1 8MHz, Q2 32.768kHz, Q3 BC817-40SMD, U1 USBUF02W6

Commit message: update circuit
Connect GPIOA 10 to NC pin, using pwm
Connections:
- net PA10: now also JP1.3
Routing:
- net PA10: track 13.4 -> 35.1 mm, vias 2 -> 3
- net PB13: track 27.4 -> 25.4 mm
- net PB15: track 28.3 -> 26.2 mm
- net PB14: track 24.7 -> 22.6 mm
- net PB12: track 23.9 -> 21.8 mm
- net PA8: track 24.9 -> 23.7 mm
