File: Eagle/rev. D/IRQF103C8revC.sch (EAGLE design)
At the start: 68 parts, among them IC1 STM32F10XCXT6, IC2 LM1117IMPX-3.3, IC3 LM1117MPX-5.0, Q1 8MHz, Q2 32.768kHz, Q3 BC817-40SMD, U1 USBUF02W6

Commit message: update circuit
Connect GPIOA 10 to NC pin, using pwm
Connections:
- net PA10: now also JP1.3
Changed lines of the file:
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@@
 <drawing>
 <settings>
-<setting alwaysvectorfont="no"/>
+<setting alwaysvectorfont="yes"/>
 <setting keepoldvectorfont="yes"/>
 <setting verticaltext="up"/>
@@
 <label x="317.5" y="114.3" size="1.778" layer="95" rot="R270" xref="yes"/>
 </segment>
+<segment>
+<pinref part="JP1" gate="A" pin="3"/>
+<wire x1="154.94" y1="99.06" x2="139.7" y2="99.06" width="0.1524" layer="91"/>
+<label x="139.7" y="99.06" size="1.778" layer="95" rot="R180" xref="yes"/>
+</segment>
 </net>
 <net name="PA9" class="0">
@@
 </segment>
 <segment>
+<pinref part="JP1" gate="A" pin="4"/>
+<wire x1="162.56" y1="99.06" x2="180.34" y2="99.06" width="0.1524" layer="91"/>
 <label x="180.34" y="99.06" size="1.778" layer="95" xref="yes"/>
-<wire x1="162.56" y1="99.06" x2="180.34" y2="99.06" width="0.1524" layer="91"/>
-<pinref part="JP1" gate="A" pin="4"/>
-</segment>
-</net>
+</segment>
+</net>
